Commit message: [1.2.0] Added sensor plugins
Extended the URDF model with Xacro calls to include Gazebo sensor plugins.

Signed-off-by: Helio Perroni Filho <xperroni@gmail.com>

File: urdf/roselito.xacro (robot description, xacro)
@@ -6,44 +6,15 @@
 <robot name="roselito" xmlns:xacro="http://www.ros.org/wiki/xacro">
   <xacro:include filename="$(find roselito_description)/urdf/roselito.xacro"/>
-  <xacro:macro
-    name="add_controller"
-    params="position"
-  >
-    <gazebo>
-      <plugin name="wheels_${position}_controller" filename="libgazebo_ros_diff_drive.so">
-        <update_rate>50</update_rate>
-        <left_joint>joint_wheel_${position}_left</left_joint>
-        <right_joint>joint_wheel_${position}_right</right_joint>
-        <wheel_separation>${wheel_separation}</wheel_separation>
-        <wheel_diameter>${wheel_diameter}</wheel_diameter>
-        <max_wheel_torque>20</max_wheel_torque>
-        <max_wheel_acceleration>1.0</max_wheel_acceleration>
-        <command_topic>cmd_vel</command_topic>
-        <odometry_topic>odom</odometry_topic>
-        <odometry_frame>odom</odometry_frame>
-        <robot_base_frame>base_link</robot_base_frame>
-        <publish_odom>true</publish_odom>
-        <publish_odom_tf>true</publish_odom_tf>
-        <publish_wheel_tf>false</publish_wheel_tf>
-        <publish_wheel_joint_state>true</publish_wheel_joint_state>
-      </plugin>
-    </gazebo>
-  </xacro:macro>
-  <!-- See: http://sdformat.org/tutorials?tut=sdformat_urdf_extensions&cat=specification -->
-  <xacro:macro
-    name="remove_friction"
-    params="position"
-  >
-    <gazebo reference="wheel_${position}_left">
-      <mu1>0.0</mu1>
-      <mu2>0.0</mu2>
-    </gazebo>
-    <gazebo reference="wheel_${position}_right">
-      <mu1>0.0</mu1>
-      <mu2>0.0</mu2>
-    </gazebo>
-  </xacro:macro>
-  <xacro:add_controller position="center"/>
+  <xacro:include filename="$(find ros_commons)/urdf/gazebo.xacro"/>
+  <xacro:differential_controller
+    name="wheels_center"
+    left_joint="joint_wheel_center_left"
+    right_joint="joint_wheel_center_right"
+    wheel_separation="${wheel_separation}"
+    wheel_diameter="${wheel_diameter}"
+  />
   <xacro:remove_friction position="front"/>
   <xacro:remove_friction position="rear"/>
+  <xacro:depth_camera name="camera_front"/>
+  <xacro:lidar_2d name="laser"/>
 </robot>

Commit message: [1.2.1] Proper updating wheel joint states
Use of joint_state_publisher to set fixed joint states for wheels created
problems with RViz. Fixed by using Gazebo plugins to generate joint state
updates for all wheels.

Signed-off-by: Helio Perroni Filho <xperroni@gmail.com>

File: urdf/roselito.xacro (robot description, xacro)
@@ -7,11 +7,21 @@
   <xacro:include filename="$(find roselito_description)/urdf/roselito.xacro"/>
   <xacro:include filename="$(find ros_commons)/urdf/gazebo.xacro"/>
-  <xacro:differential_controller
-    name="wheels_center"
-    left_joint="joint_wheel_center_left"
-    right_joint="joint_wheel_center_right"
-    wheel_separation="${wheel_separation}"
-    wheel_diameter="${wheel_diameter}"
-  />
+  <xacro:macro
+    name="add_controller"
+    params="
+      position
+    "
+  >
+    <xacro:differential_controller
+      name="wheels_${position}"
+      left_joint="joint_wheel_${position}_left"
+      right_joint="joint_wheel_${position}_right"
+      wheel_separation="${wheel_separation}"
+      wheel_diameter="${wheel_diameter}"
+    />
+  </xacro:macro>
+  <xacro:add_controller position="front"/>
+  <xacro:add_controller position="center"/>
+  <xacro:add_controller position="rear"/>
   <xacro:remove_friction position="front"/>
   <xacro:remove_friction position="rear"/>

Commit message: [1.3.0] Skid steering Gazebo plugin
Used a new macro to have a single differential drive plugin control all six
wheels in the robot.

Signed-off-by: Helio Perroni Filho <xperroni@gmail.com>

File: urdf/roselito.xacro (robot description, xacro)
@@ -8,22 +8,38 @@
   <xacro:include filename="$(find ros_commons)/urdf/gazebo.xacro"/>
   <xacro:macro
-    name="add_controller"
+    name="wheel_joint_names"
     params="
       position
-      publish_odom:=false
     "
   >
-    <xacro:differential_controller
-      name="wheels_${position}"
-      left_joint="joint_wheel_${position}_left"
-      right_joint="joint_wheel_${position}_right"
-      wheel_separation="${wheel_separation}"
-      wheel_diameter="${wheel_diameter}"
-      publish_odom="${publish_odom}"
-    />
+    <joint_name>joint_wheel_${position}_left</joint_name>
+    <joint_name>joint_wheel_${position}_right</joint_name>
   </xacro:macro>
-  <xacro:add_controller position="front"/>
-  <xacro:add_controller position="center" publish_odom="true"/>
-  <xacro:add_controller position="rear"/>
+  <xacro:macro
+    name="wheel_attributes"
+    params="
+      position
+    "
+  >
+    <left_joint>joint_wheel_${position}_left</left_joint>
+    <right_joint>joint_wheel_${position}_right</right_joint>
+    <wheel_diameter>${wheel_diameter}</wheel_diameter>
+    <wheel_separation>${wheel_separation}</wheel_separation>
+  </xacro:macro>
+  <xacro:skid_controller
+    name="wheels"
+  >
+    <joints>
+      <xacro:wheel_joint_names position="front"/>
+      <xacro:wheel_joint_names position="center"/>
+      <xacro:wheel_joint_names position="rear"/>
+    </joints>
+    <wheels>
+      <num_wheel_pairs>3</num_wheel_pairs>
+      <xacro:wheel_attributes position="front"/>
+      <xacro:wheel_attributes position="center"/>
+      <xacro:wheel_attributes position="rear"/>
+    </wheels>
+  </xacro:skid_controller>
   <xacro:remove_friction position="front"/>
   <xacro:remove_friction position="rear"/>
